File: hardware/PowerSupply.kicad_sch (KiCad schematic)
At the start: 7 parts, among them J1 Battery, J2 3.3V 500mA Regulator, J3 5.0V 500mA Regulator, J4 12V Boost Regulator

Commit message: First revision of the shield PCB
I have a few more tweaks that I would like to make before I send this
off to be manufactured. I ended up going with a 4 layer board as it has
signal wires going all over the place since I was a bit contrained with
part placement by most of the Arduino signal pins being on the right
side of the board and wanting to place connectors on the side closest
to the part to which they connect.
Parts:
- D1: symbol Device:D_Schottky -> Device:D_Schottky_AAK
Connections:
- net +BATT: now also D1.1 (A)
- net at C1.1, J2.2 (Pin_2), J3.2 (Pin_2)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: now also D1.3 (K); no longer D1.1 (K)
- net VCC: now reaches J1.2 (Pin_2), S1.2 (Com)
Changed lines of the file:
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@@
   (junction (at 137.16 67.31) (diameter 0) (color 0 0 0 0)
   )
+  (junction (at 96.52 69.85) (diameter 0) (color 0 0 0 0)
+  )
   (junction (at 151.13 135.382) (diameter 0) (color 0 0 0 0)
   )
@@
   )
   (junction (at 156.21 103.632) (diameter 0) (color 0 0 0 0)
+  )
+  (junction (at 99.06 69.85) (diameter 0) (color 0 0 0 0)
   )
   (junction (at 114.3 67.31) (diameter 0) (color 0 0 0 0)
@@
   (no_connect (at 91.44 67.31))
   (no_connect (at 142.24 101.092))
+  (wire (pts (xy 119.38 67.31) (xy 120.65 67.31))
+    (stroke (width 0) (type default) (color 0 0 0 0))
+  )
   (wire (pts (xy 114.3 62.23) (xy 114.3 67.31))
     (stroke (width 0) (type default) (color 0 0 0 0))
@@
     (stroke (width 0) (type default) (color 0 0 0 0))
   )
+  (wire (pts (xy 96.52 62.23) (xy 96.52 69.85))
+    (stroke (width 0) (type default) (color 0 0 0 0))
+  )
   (wire (pts (xy 144.78 101.092) (xy 144.78 103.632))
     (stroke (width 0) (type default) (color 0 0 0 0))
@@
     (stroke (width 0) (type default) (color 0 0 0 0))
   )
+  (wire (pts (xy 119.38 69.85) (xy 119.38 67.31))
+    (stroke (width 0) (type default) (color 0 0 0 0))
+  )
   (wire (pts (xy 111.76 67.31) (xy 114.3 67.31))
     (stroke (width 0) (type default) (color 0 0 0 0))
   )
-  (wire (pts (xy 91.44 69.85) (xy 101.6 69.85))
+  (wire (pts (xy 91.44 69.85) (xy 96.52 69.85))
     (stroke (width 0) (type default) (color 0 0 0 0))
   )
@@
     (stroke (width 0) (type default) (color 0 0 0 0))
   )
-  (wire (pts (xy 93.98 61.468) (xy 93.98 72.39))
+  (wire (pts (xy 93.98 62.23) (xy 93.98 72.39))
     (stroke (width 0) (type default) (color 0 0 0 0))
   )
@@
     (stroke (width 0) (type default) (color 0 0 0 0))
   )
+  (wire (pts (xy 99.06 62.23) (xy 99.06 69.85))
+    (stroke (width 0) (type default) (color 0 0 0 0))
+  )
+  (wire (pts (xy 96.52 69.85) (xy 99.06 69.85))
+    (stroke (width 0) (type default) (color 0 0 0 0))
+  )
   (wire (pts (xy 93.98 72.39) (xy 93.98 74.93))
     (stroke (width 0) (type default) (color 0 0 0 0))
@@
     (stroke (width 0) (type default) (color 0 0 0 0))
   )
+  (wire (pts (xy 120.65 69.85) (xy 119.38 69.85))
+    (stroke (width 0) (type default) (color 0 0 0 0))
+  )
   (wire (pts (xy 156.21 96.012) (xy 156.21 103.632))
     (stroke (width 0) (type default) (color 0 0 0 0))
@@
     (stroke (width 0) (type default) (color 0 0 0 0))
   )
-  (wire (pts (xy 119.38 67.31) (xy 121.92 67.31))
-    (stroke (width 0) (type default) (color 0 0 0 0))
-  )
   (wire (pts (xy 129.54 67.31) (xy 132.08 67.31))
     (stroke (width 0) (type default) (color 0 0 0 0))
@@
   )
   (wire (pts (xy 160.02 58.42) (xy 160.02 67.31))
+    (stroke (width 0) (type default) (color 0 0 0 0))
+  )
+  (wire (pts (xy 99.06 69.85) (xy 101.6 69.85))
     (stroke (width 0) (type default) (color 0 0 0 0))
   )
@@
     )
     (property "Datasheet" "" (id 3) (at 156.21 96.012 0)
+      (effects (font (size 1.27 1.27)) hide)
+    )
+    (pin "1")
+  )
+  (symbol (lib_id "power:PWR_FLAG") (at 96.52 62.23 0) (unit 1)
+    (in_bom yes) (on_board yes) (fields_autoplaced)
+    (property "Reference" "#FLG06" (id 0) (at 96.52 60.325 0)
+      (effects (font (size 1.27 1.27)) hide)
+    )
+    (property "Value" "PWR_FLAG" (id 1) (at 96.52 57.15 0)
+      (effects (font (size 1.27 1.27)) hide)
+    )
+    (property "Footprint" "" (id 2) (at 96.52 62.23 0)
+      (effects (font (size 1.27 1.27)) hide)
+    )
+    (property "Datasheet" "~" (id 3) (at 96.52 62.23 0)
       (effects (font (size 1.27 1.27)) hide)
     )
@@
     (pin "1")
   )
-  (symbol (lib_id "power:PWR_FLAG") (at 93.98 61.468 0) (unit 1)
-    (in_bom yes) (on_board yes) (fields_autoplaced)
-    (property "Reference" "#FLG01" (id 0) (at 93.98 59.563 0)
-      (effects (font (size 1.27 1.27)) hide)
-    )
-    (property "Value" "PWR_FLAG" (id 1) (at 93.98 56.388 0)
-      (effects (font (size 1.27 1.27)) hide)
-    )
-    (property "Footprint" "" (id 2) (at 93.98 61.468 0)
-      (effects (font (size 1.27 1.27)) hide)
-    )
-    (property "Datasheet" "~" (id 3) (at 93.98 61.468 0)
+  (symbol (lib_id "power:PWR_FLAG") (at 93.98 62.23 0) (unit 1)
+    (in_bom yes) (on_board yes) (fields_autoplaced)
+    (property "Reference" "#FLG01" (id 0) (at 93.98 60.325 0)
+      (effects (font (size 1.27 1.27)) hide)
+    )
+    (property "Value" "PWR_FLAG" (id 1) (at 93.98 57.15 0)
+      (effects (font (size 1.27 1.27)) hide)
+    )
+    (property "Footprint" "" (id 2) (at 93.98 62.23 0)
+      (effects (font (size 1.27 1.27)) hide)
+    )
+    (property "Datasheet" "~" (id 3) (at 93.98 62.23 0)
       (effects (font (size 1.27 1.27)) hide)
     )
@@
     )
     (property "Datasheet" "" (id 3) (at 160.02 127.762 0)
+      (effects (font (size 1.27 1.27)) hide)
+    )
+    (pin "1")
+  )
+  (symbol (lib_id "power:VCC") (at 99.06 62.23 0) (unit 1)
+    (in_bom yes) (on_board yes) (fields_autoplaced)
+    (property "Reference" "#PWR026" (id 0) (at 99.06 66.04 0)
+      (effects (font (size 1.27 1.27)) hide)
+    )
+    (property "Value" "VCC" (id 1) (at 99.06 57.15 0))
+    (property "Footprint" "" (id 2) (at 99.06 62.23 0)
+      (effects (font (size 1.27 1.27)) hide)
+    )
+    (property "Datasheet" "" (id 3) (at 99.06 62.23 0)
       (effects (font (size 1.27 1.27)) hide)
     )
@@
     (pin "6")
   )
-  (symbol (lib_id "Device:D_Schottky") (at 125.73 67.31 180) (unit 1)
+  (symbol (lib_id "Device:D_Schottky_AAK") (at 125.73 67.31 180) (unit 1)
     (in_bom yes) (on_board yes)
     (property "Reference" "D1" (id 0) (at 125.984 64.262 0))
@@
     (pin "1")
     (pin "2")
+    (pin "3")
   )
   (symbol (lib_id "Connector_Generic:Conn_01x04") (at 142.24 59.69 90) (unit 1)

Commit message: Cleanup PCB layout
* Made the board outline a bit smaller.
* Added the 3D .step files for all of the parts that I could find. This
  was all the parts except for the IMU from Adafruit.
* Fixed an issue where I had the back distance sensors facing in the
  wrong direction.
* Added CC BY-SA licensing info for the KiCad design files.
Other:
- title: (none) -> RugRover Shield
Changed lines of the file:
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@@
 (kicad_sch (version 20211123) (generator eeschema)
   (paper "A")
+  (title_block
+    (title "RugRover Shield")
+    (rev "0.1")
+    (comment 1 "CC BY-SA 4.0")
+  )
   (junction (at 119.38 67.31) (diameter 0) (color 0 0 0 0)
   )
