File: hardware/Motors.kicad_sch (KiCad schematic)
At the start: 8 parts, among them J22 LMotor-1, J23 RMotor-1, J24 LMotor-2, J25 RMotor-2, J26 LeftMotor Conn, J27 RightMotor Conn

Commit message: First revision of the shield PCB
I have a few more tweaks that I would like to make before I send this
off to be manufactured. I ended up going with a 4 layer board as it has
signal wires going all over the place since I was a bit contrained with
part placement by most of the Arduino signal pins being on the right
side of the board and wanting to place connectors on the side closest
to the part to which they connect.
Parts:
- J26, J27: footprint Connector_PinSocket_2.54mm:PinSocket_1x06_P2.54mm_Vertical -> Connector_PinSocket_2.54mm:PinSocket_1x06_P2.54mm_Horizontal
Changed lines of the file:
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@@
       (effects (font (size 1.27 1.27)) (justify left))
     )
-    (property "Footprint" "Connector_PinSocket_2.54mm:PinSocket_1x06_P2.54mm_Vertical" (id 2) (at 186.69 118.11 0)
+    (property "Footprint" "Connector_PinSocket_2.54mm:PinSocket_1x06_P2.54mm_Horizontal" (id 2) (at 186.69 118.11 0)
       (effects (font (size 1.27 1.27)) hide)
     )
@@
       (effects (font (size 1.27 1.27)) (justify left))
     )
-    (property "Footprint" "Connector_PinSocket_2.54mm:PinSocket_1x06_P2.54mm_Vertical" (id 2) (at 186.69 72.39 0)
+    (property "Footprint" "Connector_PinSocket_2.54mm:PinSocket_1x06_P2.54mm_Horizontal" (id 2) (at 186.69 72.39 0)
       (effects (font (size 1.27 1.27)) hide)
     )

Commit message: Cleanup PCB layout
* Made the board outline a bit smaller.
* Added the 3D .step files for all of the parts that I could find. This
  was all the parts except for the IMU from Adafruit.
* Fixed an issue where I had the back distance sensors facing in the
  wrong direction.
* Added CC BY-SA licensing info for the KiCad design files.
Other:
- title: (none) -> RugRover Shield
Changed lines of the file:
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@@
   (paper "A")
   (title_block
+    (title "RugRover Shield")
     (date "2022-03-29")
     (rev "0.1")
+    (comment 1 "CC BY-SA 4.0")
   )
   (junction (at 110.49 113.03) (diameter 0) (color 0 0 0 0)

Commit message: Re-align schematic to PCB
While laying out the PCB, I modified the footprints used for the
headers connecting to the nRF52-DK and changed some of the header value
names. This commit makes the same updates to the schematic sheets.
Parts:
- J26: value LeftMotor Conn -> Left Motor
- J27: value RightMotor Conn -> Right Motor
Changed lines of the file:
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@@
       (effects (font (size 1.27 1.27)) (justify left))
     )
-    (property "Value" "RightMotor Conn" (id 1) (at 178.8668 128.6764 0)
+    (property "Value" "Right Motor" (id 1) (at 178.8668 128.6764 0)
       (effects (font (size 1.27 1.27)) (justify left))
     )
@@
       (effects (font (size 1.27 1.27)) (justify left))
     )
-    (property "Value" "LeftMotor Conn" (id 1) (at 179.2732 83.0072 0)
+    (property "Value" "Left Motor" (id 1) (at 179.2732 83.0072 0)
       (effects (font (size 1.27 1.27)) (justify left))
     )
