File: hardware/shield.kicad_sch (KiCad schematic)
At the start: 11 parts, among them P11 CONN_01X01, P12 CONN_01X01, P2 Power, P3 Analog, P5 GPIO, P6 GPIO, P7 GPIO, P8 CONN_01X01, P9 CONN_01X01

Commit message: Add note about P0.9 & P0.10 and NFC
These two pins are used for the encoders but require special code to
make them available as GPIO and the nRF52-DK also needs to be modified
to remove the 0 ohm R25/R26 resistors and place them on on R27/R28
instead to move the connection from the NFC antenna to the headers on
the development kit which connect to my shield.
Other:
- note added: "P0.9 and P0.10 default to NFC antenna. Requires UICR and R25/R26 changes to use as GPIO."
Changed lines of the file:
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@@
     (effects (font (size 1.27 1.27)) (justify right bottom))
+  )
+  (text "P0.9 and P0.10 \ndefault to NFC \nantenna. Requires \nUICR and R25/R26 \nchanges to use as\nGPIO."
+    (at 166.37 114.3 0)
+    (effects (font (size 1.27 1.27)) (justify left bottom))
   )
   (text "P0.17" (at 147.32 81.28 180)

Commit message: Update schematic to use correct pin for LMOTOR_PWM1
Other:
- note added: "P0.21"
Changed lines of the file:
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@@
     (effects (font (size 1.27 1.27)) (justify left bottom))
   )
-  (text "P0.2" (at 141.986 118.11 0)
+  (text "P0.21" (at 141.986 118.11 0)
     (effects (font (size 1.27 1.27)) (justify left bottom))
   )
